Commit message: lidar support and follower tuning

File: my_robot/urdf/my_robot.xacro (robot description, xacro)
@@ -31,58 +31,90 @@
       </geometry>
     </visual>
-    <collision name='front_caster_collision'>
-      <origin xyz="0.15 0 -0.025" rpy=" 0 0 0"/>
-      <geometry>
-        <sphere radius="0.025"/>
-      </geometry>
-    </collision>
-    <visual name='front_caster_visual'>
-      <origin xyz="0.15 0 -0.025" rpy=" 0 0 0"/>
-      <geometry>
-        <sphere radius="0.025"/>
-      </geometry>
-    </visual>
-  </link>
-  <link name="left_wheel">
-	<inertial>
-	  <origin xyz="0 0 0" rpy=" 0 1.5707 1.5707"/>
-	  <mass value="2"/>
-	  <inertia
-		  ixx="0.1" ixy="0" ixz="0"
-    		  iyy="0.1" iyz="0"
-    		  izz="0.1"/>
-	</inertial>
-	<collision>
-	  <origin xyz="0 0 0" rpy=" 0 1.5707 1.5707"/>
-	  <geometry>
-		  <cylinder radius="0.07" length="0.05"/>
-	  </geometry>
-	</collision>
-	<visual>
-	  <origin xyz="0 0 0" rpy=" 0 1.5707 1.5707"/>
-	  <geometry>
-		  <cylinder radius="0.07" length="0.05"/>
-	  </geometry>
-	</visual>
-  </link>
-  <link name="right_wheel">
-	<inertial>
-	  <origin xyz="0 0 0" rpy=" 0 1.5707 1.5707"/>
-	  <mass value="2"/>
-	  <inertia
-		  ixx="0.1" ixy="0" ixz="0"
-    		  iyy="0.1" iyz="0"
-    		  izz="0.1"/>
-	</inertial>
-	<collision>
-	  <origin xyz="0 0 0" rpy=" 0 1.5707 1.5707"/>
-	  <geometry>
-		  <cylinder radius="0.07" length="0.05"/>
-	  </geometry>
-	</collision>
-	<visual>
-	  <origin xyz="0 0 0" rpy=" 0 1.5707 1.5707"/>
-	  <geometry>
-		  <cylinder radius="0.07" length="0.05"/>
+  </link>
+  <link name="left_wheel_back">
+	<inertial>
+	  <origin xyz="0 0 0" rpy=" 0 1.5707 1.5707"/>
+	  <mass value="2"/>
+	  <inertia
+		  ixx="0.1" ixy="0" ixz="0"
+    		  iyy="0.1" iyz="0"
+    		  izz="0.1"/>
+	</inertial>
+	<collision>
+	  <origin xyz="0 0 0" rpy=" 0 1.5707 1.5707"/>
+	  <geometry>
+		  <cylinder radius="0.07" length="0.03"/>
+	  </geometry>
+	</collision>
+	<visual>
+	  <origin xyz="0 0 0" rpy=" 0 1.5707 1.5707"/>
+	  <geometry>
+		  <cylinder radius="0.07" length="0.03"/>
+	  </geometry>
+	</visual>
+  </link>
+  <link name="right_wheel_back">
+	<inertial>
+	  <origin xyz="0 0 0" rpy=" 0 1.5707 1.5707"/>
+	  <mass value="2"/>
+	  <inertia
+		  ixx="0.1" ixy="0" ixz="0"
+    		  iyy="0.1" iyz="0"
+    		  izz="0.1"/>
+	</inertial>
+	<collision>
+	  <origin xyz="0 0 0" rpy=" 0 1.5707 1.5707"/>
+	  <geometry>
+		  <cylinder radius="0.07" length="0.03"/>
+	  </geometry>
+	</collision>
+	<visual>
+	  <origin xyz="0 0 0" rpy=" 0 1.5707 1.5707"/>
+	  <geometry>
+		  <cylinder radius="0.07" length="0.03"/>
+	  </geometry>
+	</visual>
+  </link>
+    <link name="left_wheel_front">
+	<inertial>
+	  <origin xyz="0 0 0" rpy=" 0 1.5707 1.5707"/>
+	  <mass value="2"/>
+	  <inertia
+		  ixx="0.1" ixy="0" ixz="0"
+    		  iyy="0.1" iyz="0"
+    		  izz="0.1"/>
+	</inertial>
+	<collision>
+	  <origin xyz="0 0 0" rpy=" 0 1.5707 1.5707"/>
+	  <geometry>
+		  <cylinder radius="0.07" length="0.03"/>
+	  </geometry>
+	</collision>
+	<visual>
+	  <origin xyz="0 0 0" rpy=" 0 1.5707 1.5707"/>
+	  <geometry>
+		  <cylinder radius="0.07" length="0.03"/>
+	  </geometry>
+	</visual>
+  </link>
+  <link name="right_wheel_front">
+	<inertial>
+	  <origin xyz="0 0 0" rpy=" 0 1.5707 1.5707"/>
+	  <mass value="2"/>
+	  <inertia
+		  ixx="0.1" ixy="0" ixz="0"
+    		  iyy="0.1" iyz="0"
+    		  izz="0.1"/>
+	</inertial>
+	<collision>
+	  <origin xyz="0 0 0" rpy=" 0 1.5707 1.5707"/>
+	  <geometry>
+		  <cylinder radius="0.07" length="0.03"/>
+	  </geometry>
+	</collision>
+	<visual>
+	  <origin xyz="0 0 0" rpy=" 0 1.5707 1.5707"/>
+	  <geometry>
+		  <cylinder radius="0.07" length="0.03"/>
 	  </geometry>
 	</visual>
@@ -135,15 +167,53 @@
   	</collision>
   </link>
-  <joint type="continuous" name="left_wheel_hinge">
-    <origin xyz="-0.25 0.2 0" rpy="0 0 0"/>
-    <child link="left_wheel"/>
-    <parent link="chassis"/>
-    <axis xyz="0 1 0" rpy="0 0 0"/>
-    <limit effort="10000" velocity="1000"/>
-    <dynamics damping="1.0" friction="1.0"/>
-  </joint>
-  <joint type="continuous" name="right_wheel_hinge">
-    <origin xyz="-0.25 -0.2 0" rpy="0 0 0"/>
-    <child link="right_wheel"/>
+  <link name="lidar_support">
+  	<inertial>
+  	  <origin xyz="0 0 0" rpy=" 0 0 0"/>
+	  <mass value="0.1"/>
+	  <inertia
+		  ixx="1e-6" ixy="0" ixz="0"
+    		  iyy="1e-6" iyz="0"
+    		  izz="1e-6"/>
+  	</inertial>
+  	<visual>
+  	  <origin xyz="0 0 0" rpy=" 0 0 0"/>
+  	  <geometry>
+  	  	<box size="0.03 0.03 0.10"/>
+  	  </geometry>
+  	</visual>
+  	<collision>
+  	  <origin xyz="0 0 0" rpy=" 0 0 0"/>
+  	  <geometry>
+  	  	<box size="0.03 0.03 0.10"/>
+  	  </geometry>
+  	</collision>
+  </link>
+  <joint type="continuous" name="left_wheel_back_hinge">
+    <origin xyz="-0.25 0.2 0.0" rpy="0 0 0"/>
+    <child link="left_wheel_back"/>
+    <parent link="chassis"/>
+    <axis xyz="0 1 0" rpy="0 0 0"/>
+    <limit effort="10000" velocity="1000"/>
+    <dynamics damping="1.0" friction="1.0"/>
+  </joint>
+  <joint type="continuous" name="right_wheel_back_hinge">
+    <origin xyz="-0.25 -0.2 0.0" rpy="0 0 0"/>
+    <child link="right_wheel_back"/>
+    <parent link="chassis"/>
+    <axis xyz="0 1 0" rpy="0 0 0"/>
+    <limit effort="10000" velocity="1000"/>
+    <dynamics damping="1.0" friction="1.0"/>
+  </joint>
+  <joint type="continuous" name="left_wheel_front_hinge">
+    <origin xyz="0.25 0.2 0.0" rpy="0 0 0"/>
+    <child link="left_wheel_front"/>
+    <parent link="chassis"/>
+    <axis xyz="0 1 0" rpy="0 0 0"/>
+    <limit effort="10000" velocity="1000"/>
+    <dynamics damping="1.0" friction="1.0"/>
+  </joint>
+  <joint type="continuous" name="right_wheel_front_hinge">
+    <origin xyz="0.25 -0.2 0.0" rpy="0 0 0"/>
+    <child link="right_wheel_front"/>
     <parent link="chassis"/>
     <axis xyz="0 1 0" rpy="0 0 0"/>
@@ -152,19 +222,31 @@
   </joint>
   <joint type="fixed" name="camera_joint">
-    <origin xyz="0.25 0 0" rpy="0 0 0"/>
+    <origin xyz="0.3 0 0" rpy="0 0 0"/>
     <child link="camera"/>
     <parent link="chassis"/>
     <axis xyz="0 1 0" rpy="0 0 0"/>
   </joint>
+  <joint type="fixed" name="support_joint">
+    <origin xyz="0.15 0 0.05" rpy="0 0 0"/>
+    <child link="lidar_support"/>
+    <parent link="chassis"/>
+    <axis xyz="0 1 0" rpy="0 0 0"/>
+  </joint>
   <joint type="fixed" name="hokuyo_joint">
-    <origin xyz="0.15 0 0.1" rpy="0 0 0"/>
+    <origin xyz="0 0 0.10" rpy="0 0 0"/>
     <child link="hokuyo"/>
-    <parent link="chassis"/>
-    <axis xyz="0 1 0" rpy="0 0 0"/>
-  </joint>
- <gazebo reference="left_wheel">
-    <material>Gazebo/Black</material>
- </gazebo>
- <gazebo reference="right_wheel">
+    <parent link="lidar_support"/>
+    <axis xyz="0 1 0" rpy="0 0 0"/>
+  </joint>
+ <gazebo reference="left_wheel_back">
+    <material>Gazebo/Black</material>
+ </gazebo>
+ <gazebo reference="right_wheel_back">
+    <material>Gazebo/Black</material>
+ </gazebo>
+  <gazebo reference="left_wheel_front">
+    <material>Gazebo/Black</material>
+ </gazebo>
+ <gazebo reference="right_wheel_front">
     <material>Gazebo/Black</material>
  </gazebo>
